File: MiniProj.kicad_pcb (KiCad board)
At the start: 2 copper layers, 22 parts, among them SW1_UP1 SW_Push_Dual, SW2_DOWN1 SW_Push_Dual, SW3_LEFT1 SW_Push_Dual, SW4_RIGHT1 SW_Push_Dual, SW5_RESET1 SW_Push_Dual, U1 STM32F051R8Tx

Commit message: df
df
Parts:
- added J1: 1935161, digikey-footprints:Terminal_Block_D1.3mm_P5mm, F.Cu at (281.9, 16.5)
- added PS1: IA0503S_copy, PDS1-S3-S3-M_1:CONV_PDS1-S3-S3-M, F.Cu at (268.0, 19.1)
- moved C5 35.5 mm to (259.1, 17.8), turned to 270 degrees
- moved C6 25.4 mm to (256.5, 17.8), turned to 270 degrees
- moved R3 14.4 mm to (195.4, 63.9)
- moved R4 14.4 mm to (196.8, 59.7)
- moved R6 13.2 mm to (160.0, 56.7)
- moved C2 11.4 mm to (190.5, 68.6)
- moved R5 10.2 mm to (154.9, 54.6)
- moved C1 10.2 mm to (196.8, 39.4)
- moved C3 10.2 mm to (157.5, 62.2)
- moved C4 10.2 mm to (219.7, 59.7)
- moved C7 10.2 mm to (210.8, 19.1)
- moved R2 10.2 mm to (196.8, 35.6)
- moved R7 10.2 mm to (217.2, 52.1)
- moved R8 10.2 mm to (219.2, 55.9)
- moved R9 10.2 mm to (210.8, 15.7), turned to 0 degrees
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Connections:
- R1 pad 2: +3V0 -> VDD
- R4 pad 2: +3V0 -> VDD
- R5 pad 2: +3V0 -> VDD
- R7 pad 2: +3V0 -> VDD
Routing:
- net VDD: track 0.00 -> 292.5 mm, vias 0 -> 9
- net GND: track 0.00 -> 284.7 mm, vias 0 -> 7
- net PC2: track 0.00 -> 92.6 mm, vias 0 -> 2
- net PC1: track 0.00 -> 72.5 mm, vias 0 -> 1
- net PC3: track 0.00 -> 42.5 mm
- net PC0: track 0.00 -> 41.4 mm
- net NRST: track 0.00 -> 33.6 mm, vias 0 -> 2
- net Net-(R7-Pad1): track 0.00 -> 25.4 mm
- net Net-(R5-Pad1): track 0.00 -> 23.8 mm, vias 0 -> 1
- net Net-(R3-Pad2): track 0.00 -> 21.5 mm
- net Net-(R1-Pad1): track 0.00 -> 21.1 mm
- net GNDREF: track 0.00 -> 11.3 mm
- net +5V: track 0.00 -> 9.48 mm
