File: MiniProj.sch (KiCad schematic (older format))
At the start: 22 parts, among them SW1_UP1 SW_Push_Dual, SW2_DOWN1 SW_Push_Dual, SW3_LEFT1 SW_Push_Dual, SW4_RIGHT1 SW_Push_Dual, SW5_RESET1 SW_Push_Dual, U1 STM32F051R8Tx

Commit message: Add files via upload
Parts:
- added PS?: IA0305S, Converter_DCDC:Converter_DCDC_XP_POWER-IAxxxxS_THT, symbol Converter_DCDC:IA0305S
- C1, C2, C3, C4, C6, C7: footprint (none) -> Capacitor_SMD:C_0201_0603Metric
- C5: footprint (none) -> Capacitor_SMD:C_0402_1005Metric
- R1, R2, R3, R4, R5, R6, R7, R8, R9: footprint (none) -> Resistor_SMD:R_0402_1005Metric
- SW1_UP1, SW3_LEFT1, SW4_RIGHT1, SW5_RESET1: footprint (none) -> Button_Switch_THT:SW_TH_Tactile_Omron_B3F-10xx
- SW2_DOWN1: footprint Test -> Button_Switch_THT:SW_TH_Tactile_Omron_B3F-10xx
Changed lines of the file:
@@
 EESchema Schematic File Version 4
+LIBS:MiniProj-cache
 EELAYER 30 0
 EELAYER END
@@
 F 0 "C5" H 6315 1596 50  0000 L CNN
 F 1 "1uF" H 6315 1505 50  0000 L CNN
-F 2 "" H 6238 1400 50  0001 C CNN
+F 2 "Capacitor_SMD:C_0402_1005Metric" H 6238 1400 50  0001 C CNN
 F 3 "~" H 6200 1550 50  0001 C CNN
 	1    6200 1550
@@
 F 0 "C6" H 6715 1596 50  0000 L CNN
 F 1 "100nF" H 6715 1505 50  0000 L CNN
-F 2 "" H 6638 1400 50  0001 C CNN
+F 2 "Capacitor_SMD:C_0201_0603Metric" H 6638 1400 50  0001 C CNN
 F 3 "~" H 6600 1550 50  0001 C CNN
 	1    6600 1550
@@
 F 0 "SW1_UP1" V 550 1500 50  0000 C CNN
 F 1 "SW_Push_Dual" V 650 1500 50  0000 C CNN
-F 2 "" H 1000 1800 50  0001 C CNN
+F 2 "Button_Switch_THT:SW_TH_Tactile_Omron_B3F-10xx" H 1000 1800 50  0001 C CNN
 F 3 "~" H 1000 1800 50  0001 C CNN
 	1    1000 1600
@@
 F 0 "C1" H 1715 1746 50  0000 L CNN
 F 1 ".1uF" H 1715 1655 50  0000 L CNN
-F 2 "" H 1638 1550 50  0001 C CNN
+F 2 "Capacitor_SMD:C_0201_0603Metric" H 1638 1550 50  0001 C CNN
 F 3 "~" H 1600 1700 50  0001 C CNN
 	1    1600 1700
@@
 F 0 "R2" V 1143 1300 50  0000 C CNN
 F 1 "10k" V 1234 1300 50  0000 C CNN
-F 2 "" V 1280 1300 50  0001 C CNN
+F 2 "Resistor_SMD:R_0402_1005Metric" V 1280 1300 50  0001 C CNN
 F 3 "~" H 1350 1300 50  0001 C CNN
 	1    1350 1300
@@
 F 0 "R1" H 930 954 50  0000 R CNN
 F 1 "10k" H 930 1045 50  0000 R CNN
-F 2 "" V 930 1000 50  0001 C CNN
+F 2 "Resistor_SMD:R_0402_1005Metric" V 930 1000 50  0001 C CNN
 F 3 "~" H 1000 1000 50  0001 C CNN
 	1    1000 1000
@@
 F 0 "SW4_RIGHT1" V 550 7000 50  0000 C CNN
 F 1 "SW_Push_Dual" V 650 7000 50  0000 C CNN
-F 2 "" H 1000 7300 50  0001 C CNN
+F 2 "Button_Switch_THT:SW_TH_Tactile_Omron_B3F-10xx" H 1000 7300 50  0001 C CNN
 F 3 "~" H 1000 7300 50  0001 C CNN
 	1    1000 7100
@@
 F 0 "C4" H 1715 7246 50  0000 L CNN
 F 1 ".1uF" H 1715 7155 50  0000 L CNN
-F 2 "" H 1638 7050 50  0001 C CNN
+F 2 "Capacitor_SMD:C_0201_0603Metric" H 1638 7050 50  0001 C CNN
 F 3 "~" H 1600 7200 50  0001 C CNN
 	1    1600 7200
@@
 F 0 "R8" V 1143 6800 50  0000 C CNN
 F 1 "10k" V 1234 6800 50  0000 C CNN
-F 2 "" V 1280 6800 50  0001 C CNN
+F 2 "Resistor_SMD:R_0402_1005Metric" V 1280 6800 50  0001 C CNN
 F 3 "~" H 1350 6800 50  0001 C CNN
 	1    1350 6800
@@
 F 0 "R7" H 930 6454 50  0000 R CNN
 F 1 "10k" H 930 6545 50  0000 R CNN
-F 2 "" V 930 6500 50  0001 C CNN
+F 2 "Resistor_SMD:R_0402_1005Metric" V 930 6500 50  0001 C CNN
 F 3 "~" H 1000 6500 50  0001 C CNN
 	1    1000 6500
@@
 F 0 "SW3_LEFT1" V 550 5200 50  0000 C CNN
 F 1 "SW_Push_Dual" V 650 5200 50  0000 C CNN
-F 2 "" H 1000 5500 50  0001 C CNN
+F 2 "Button_Switch_THT:SW_TH_Tactile_Omron_B3F-10xx" H 1000 5500 50  0001 C CNN
 F 3 "~" H 1000 5500 50  0001 C CNN
 	1    1000 5300
@@
 F 0 "R6" V 1143 5000 50  0000 C CNN
 F 1 "10k" V 1234 5000 50  0000 C CNN
-F 2 "" V 1280 5000 50  0001 C CNN
+F 2 "Resistor_SMD:R_0402_1005Metric" V 1280 5000 50  0001 C CNN
 F 3 "~" H 1350 5000 50  0001 C CNN
 	1    1350 5000
@@
 F 0 "R5" H 930 4654 50  0000 R CNN
 F 1 "10k" H 930 4745 50  0000 R CNN
-F 2 "" V 930 4700 50  0001 C CNN
+F 2 "Resistor_SMD:R_0402_1005Metric" V 930 4700 50  0001 C CNN
 F 3 "~" H 1000 4700 50  0001 C CNN
 	1    1000 4700
@@
 F 0 "R4" H 930 2804 50  0000 R CNN
 F 1 "10k" H 930 2895 50  0000 R CNN
-F 2 "" V 930 2850 50  0001 C CNN
+F 2 "Resistor_SMD:R_0402_1005Metric" V 930 2850 50  0001 C CNN
 F 3 "~" H 1000 2850 50  0001 C CNN
 	1    1000 2850
@@
 F 0 "R3" V 1143 3150 50  0000 C CNN
 F 1 "10k" V 1234 3150 50  0000 C CNN
-F 2 "" V 1280 3150 50  0001 C CNN
+F 2 "Resistor_SMD:R_0402_1005Metric" V 1280 3150 50  0001 C CNN
 F 3 "~" H 1350 3150 50  0001 C CNN
 	1    1350 3150
@@
 F 0 "C2" H 1715 3596 50  0000 L CNN
 F 1 ".1uF" H 1715 3505 50  0000 L CNN
-F 2 "" H 1638 3400 50  0001 C CNN
+F 2 "Capacitor_SMD:C_0201_0603Metric" H 1638 3400 50  0001 C CNN
 F 3 "~" H 1600 3550 50  0001 C CNN
 	1    1600 3550
@@
 F 0 "SW2_DOWN1" V 550 3350 50  0000 C CNN
 F 1 "SW_Push_Dual" V 650 3350 50  0000 C CNN
-F 2 "Test" H 1000 3650 50  0001 C CNN
+F 2 "Button_Switch_THT:SW_TH_Tactile_Omron_B3F-10xx" H 1000 3650 50  0001 C CNN
 F 3 "~" H 1000 3650 50  0001 C CNN
 	1    1000 3450
@@
 F 0 "SW5_RESET1" V 2400 5300 50  0000 C CNN
 F 1 "SW_Push_Dual" V 2500 5300 50  0000 C CNN
-F 2 "" H 2850 5600 50  0001 C CNN
+F 2 "Button_Switch_THT:SW_TH_Tactile_Omron_B3F-10xx" H 2850 5600 50  0001 C CNN
 F 3 "~" H 2850 5600 50  0001 C CNN
 	1    2850 5400
@@
 F 0 "C3" H 1715 5446 50  0000 L CNN
 F 1 ".1uF" H 1715 5355 50  0000 L CNN
-F 2 "" H 1638 5250 50  0001 C CNN
+F 2 "Capacitor_SMD:C_0201_0603Metric" H 1638 5250 50  0001 C CNN
 F 3 "~" H 1600 5400 50  0001 C CNN
 	1    1600 5400
@@
 F 0 "C7" H 3415 5546 50  0000 L CNN
 F 1 ".1uF" H 3415 5455 50  0000 L CNN
-F 2 "" H 3338 5350 50  0001 C CNN
+F 2 "Capacitor_SMD:C_0201_0603Metric" H 3338 5350 50  0001 C CNN
 F 3 "~" H 3300 5500 50  0001 C CNN
 	1    3300 5500
@@
 F 0 "R9" H 2920 4996 50  0000 L CNN
 F 1 "100k" H 2920 4905 50  0000 L CNN
-F 2 "" V 2780 4950 50  0001 C CNN
+F 2 "Resistor_SMD:R_0402_1005Metric" V 2780 4950 50  0001 C CNN
 F 3 "~" H 2850 4950 50  0001 C CNN
 	1    2850 4950
@@
 Wire Wire Line
 	1000 6200 1000 6350
+$Comp
+L Converter_DCDC:IA0305S PS?
+U 1 1 5DDAA351
+P 7650 3200
+F 0 "PS?" H 7650 3567 50  0000 C CNN
+F 1 "IA0305S" H 7650 3476 50  0000 C CNN
+F 2 "Converter_DCDC:Converter_DCDC_XP_POWER-IAxxxxS_THT" H 6600 2950 50  0001 L CNN
+F 3 "https://www.xppower.com/pdfs/SF_IA.pdf" H 8700 2900 50  0001 L CNN
+	1    7650 3200
+	1    0    0    -1
+$EndComp
 $EndSCHEMATC

Commit message: df
df
Parts:
- removed PS?: IA0305S, Converter_DCDC:Converter_DCDC_XP_POWER-IAxxxxS_THT, symbol Converter_DCDC:IA0305S
- added J1: 1935161, digikey-footprints:Terminal_Block_D1.3mm_P5mm, symbol dk_Terminal-Blocks-Wire-to-Board:1935161
- added J2: Screw_Terminal_01x15, TerminalBlock_4Ucon:TerminalBlock_4Ucon_1x15_P3.50mm_Horizontal, symbol Connector:Screw_Terminal_01x15
- added PS1: IA0503S_copy, PDS1-S3-S3-M_1:CONV_PDS1-S3-S3-M, symbol dk_DC-DC-Converters:IA0503S_copy
Connections:
- net labels added: +5V, GNDREF
- net labels removed: +3V0
Changed lines of the file:
@@
 	1000 850  1000 700
-$Comp
-L power:+3V0 #PWR0103
-U 1 1 5DD4D878
-P 1000 700
-F 0 "#PWR0103" H 1000 550 50  0001 C CNN
-F 1 "+3V0" H 1015 873 50  0000 C CNN
-F 2 "" H 1000 700 50  0001 C CNN
-F 3 "" H 1000 700 50  0001 C CNN
-	1    1000 700
-	1    0    0    -1
-$EndComp
 $Comp
 L Switch:SW_Push_Dual SW4_RIGHT1
@@
 $EndComp
 $Comp
-L power:+3V0 #PWR0105
-U 1 1 5DD79116
-P 1000 6200
-F 0 "#PWR0105" H 1000 6050 50  0001 C CNN
-F 1 "+3V0" H 1015 6373 50  0000 C CNN
-F 2 "" H 1000 6200 50  0001 C CNN
-F 3 "" H 1000 6200 50  0001 C CNN
-	1    1000 6200
-	1    0    0    -1
-$EndComp
-$Comp
 L Switch:SW_Push_Dual SW3_LEFT1
 U 1 1 5DD7BC4C
@@
 Wire Wire Line
 	1000 4550 1000 4400
-$Comp
-L power:+3V0 #PWR0106
-U 1 1 5DD7BC79
-P 1000 4400
-F 0 "#PWR0106" H 1000 4250 50  0001 C CNN
-F 1 "+3V0" H 1015 4573 50  0000 C CNN
-F 2 "" H 1000 4400 50  0001 C CNN
-F 3 "" H 1000 4400 50  0001 C CNN
-	1    1000 4400
-	1    0    0    -1
-$EndComp
-$Comp
-L power:+3V0 #PWR0107
-U 1 1 5DD75260
-P 1000 2550
-F 0 "#PWR0107" H 1000 2400 50  0001 C CNN
-F 1 "+3V0" H 1015 2723 50  0000 C CNN
-F 2 "" H 1000 2550 50  0001 C CNN
-F 3 "" H 1000 2550 50  0001 C CNN
-	1    1000 2550
-	1    0    0    -1
-$EndComp
 $Comp
 L power:GND #PWR0108
@@
 	1000 6200 1000 6350
 $Comp
-L Converter_DCDC:IA0305S PS?
-U 1 1 5DDAA351
-P 7650 3200
-F 0 "PS?" H 7650 3567 50  0000 C CNN
-F 1 "IA0305S" H 7650 3476 50  0000 C CNN
-F 2 "Converter_DCDC:Converter_DCDC_XP_POWER-IAxxxxS_THT" H 6600 2950 50  0001 L CNN
-F 3 "https://www.xppower.com/pdfs/SF_IA.pdf" H 8700 2900 50  0001 L CNN
-	1    7650 3200
-	1    0    0    -1
-$EndComp
+L dk_DC-DC-Converters:IA0503S_copy PS1
+U 1 1 5DD39D7E
+P 7700 2850
+F 0 "PS1" H 7700 3217 50  0000 C CNN
+F 1 "IA0503S_copy" H 7700 3126 50  0000 C CNN
+F 2 "PDS1-S3-S3-M_1:CONV_PDS1-S3-S3-M" H 6650 2600 50  0001 L CNN
+F 3 "https://www.xppower.com/pdfs/SF_IA.pdf" H 8750 2550 50  0001 L CNN
+	1    7700 2850
+	1    0    0    -1
+$EndComp
+$Comp
+L power:VDD #PWR09
+U 1 1 5DD3CA20
+P 8100 2850
+F 0 "#PWR09" H 8100 2700 50  0001 C CNN
+F 1 "VDD" V 8117 2978 50  0000 L CNN
+F 2 "" H 8100 2850 50  0001 C CNN
+F 3 "" H 8100 2850 50  0001 C CNN
+	1    8100 2850
+	0    1    1    0
+$EndComp
+$Comp
+L power:VDD #PWR01
+U 1 1 5DD45639
+P 1000 700
+F 0 "#PWR01" H 1000 550 50  0001 C CNN
+F 1 "VDD" H 1017 873 50  0000 C CNN
+F 2 "" H 1000 700 50  0001 C CNN
+F 3 "" H 1000 700 50  0001 C CNN
+	1    1000 700
+	1    0    0    -1
+$EndComp
+$Comp
+L power:VDD #PWR02
+U 1 1 5DD4C8FC
+P 1000 2550
+F 0 "#PWR02" H 1000 2400 50  0001 C CNN
+F 1 "VDD" H 1017 2723 50  0000 C CNN
+F 2 "" H 1000 2550 50  0001 C CNN
+F 3 "" H 1000 2550 50  0001 C CNN
+	1    1000 2550
+	1    0    0    -1
+$EndComp
+$Comp
+L power:VDD #PWR03
+U 1 1 5DD539F7
+P 1000 4400
+F 0 "#PWR03" H 1000 4250 50  0001 C CNN
+F 1 "VDD" H 1017 4573 50  0000 C CNN
+F 2 "" H 1000 4400 50  0001 C CNN
+F 3 "" H 1000 4400 50  0001 C CNN
+	1    1000 4400
+	1    0    0    -1
+$EndComp
+$Comp
+L power:VDD #PWR04
+U 1 1 5DD5B321
+P 1000 6200
+F 0 "#PWR04" H 1000 6050 50  0001 C CNN
+F 1 "VDD" H 1017 6373 50  0000 C CNN
+F 2 "" H 1000 6200 50  0001 C CNN
+F 3 "" H 1000 6200 50  0001 C CNN
+	1    1000 6200
+	1    0    0    -1
+$EndComp
+$Comp
+L power:GND #PWR010
+U 1 1 5DD5B7FB
+P 8100 2950
+F 0 "#PWR010" H 8100 2700 50  0001 C CNN
+F 1 "GND" V 8105 2822 50  0000 R CNN
+F 2 "" H 8100 2950 50  0001 C CNN
+F 3 "" H 8100 2950 50  0001 C CNN
+	1    8100 2950
+	0    -1   -1   0
+$EndComp
+$Comp
+L dk_Terminal-Blocks-Wire-to-Board:1935161 J1
+U 1 1 5DD699C7
+P 8200 1250
+F 0 "J1" V 8291 1172 50  0000 R CNN
+F 1 "1935161" V 8200 1172 50  0000 R CNN
+F 2 "digikey-footprints:Terminal_Block_D1.3mm_P5mm" H 8400 1450 60  0001 L CNN
+F 3 "https://media.digikey.com/pdf/Data%20Sheets/Phoenix%20Contact%20PDFs/1935161.pdf" H 8400 1550 60  0001 L CNN
+F 4 "277-1667-ND" H 8400 1650 60  0001 L CNN "Digi-Key_PN"
+F 5 "1935161" H 8400 1750 60  0001 L CNN "MPN"
+F 6 "Connectors, Interconnects" H 8400 1850 60  0001 L CNN "Category"
+F 7 "Terminal Blocks - Wire to Board" H 8400 1950 60  0001 L CNN "Family"
+F 8 "https://media.digikey.com/pdf/Data%20Sheets/Phoenix%20Contact%20PDFs/1935161.pdf" H 8400 2050 60  0001 L CNN "DK_Datasheet_Link"
+F 9 "/product-detail/en/phoenix-contact/1935161/277-1667-ND/568614" H 8400 2150 60  0001 L CNN "DK_Detail_Page"
+F 10 "TERM BLK 2POS SIDE ENTRY 5MM PCB" H 8400 2250 60  0001 L CNN "Description"
+F 11 "Phoenix Contact" H 8400 2350 60  0001 L CNN "Manufacturer"
+F 12 "Active" H 8400 2450 60  0001 L CNN "Status"
+	1    8200 1250
+	0    -1   -1   0
+$EndComp
+$Comp
+L power:+5V #PWR07
+U 1 1 5DD755D6
+P 8000 1150
+F 0 "#PWR07" H 8000 1000 50  0001 C CNN
+F 1 "+5V" V 8015 1278 50  0000 L CNN
+F 2 "" H 8000 1150 50  0001 C CNN
+F 3 "" H 8000 1150 50  0001 C CNN
+	1    8000 1150
+	0    -1   -1   0
+$EndComp
+$Comp
+L power:GNDREF #PWR08
+U 1 1 5DD7710A
+P 8000 1250
+F 0 "#PWR08" H 8000 1000 50  0001 C CNN
+F 1 "GNDREF" V 8005 1122 50  0000 R CNN
+F 2 "" H 8000 1250 50  0001 C CNN
+F 3 "" H 8000 1250 50  0001 C CNN
+	1    8000 1250
+	0    1    1    0
+$EndComp
+$Comp
+L power:GNDREF #PWR06
+U 1 1 5DD78D37
+P 7300 2950
+F 0 "#PWR06" H 7300 2700 50  0001 C CNN
+F 1 "GNDREF" V 7305 2822 50  0000 R CNN
+F 2 "" H 7300 2950 50  0001 C CNN
+F 3 "" H 7300 2950 50  0001 C CNN
+	1    7300 2950
+	0    1    1    0
+$EndComp
+$Comp
+L power:+5V #PWR05
+U 1 1 5DD79B2E
+P 7300 2750
+F 0 "#PWR05" H 7300 2600 50  0001 C CNN
+F 1 "+5V" V 7315 2878 50  0000 L CNN
+F 2 "" H 7300 2750 50  0001 C CNN
+F 3 "" H 7300 2750 50  0001 C CNN
+	1    7300 2750
+	0    -1   -1   0
+$EndComp
+$Comp
+L Connector:Screw_Terminal_01x15 J2
+U 1 1 5DD92941
+P 7050 4200
+F 0 "J2" H 7130 4242 50  0000 L CNN
+F 1 "Screw_Terminal_01x15" H 7130 4151 50  0000 L CNN
+F 2 "TerminalBlock_4Ucon:TerminalBlock_4Ucon_1x15_P3.50mm_Horizontal" H 7050 4200 50  0001 C CNN
+F 3 "~" H 7050 4200 50  0001 C CNN
+	1    7050 4200
+	1    0    0    -1
+$EndComp
